File: encoder.kicad_sch (KiCad schematic)
At the start: 42 parts

Commit message: completed and annotated schematic, passed ERC
Parts:
- added C58: 100n, symbol tbc:GCJ188R71H104KA12D
- gave numbers to parts that had none: 42
Connections:
- net +3V3: now also U7.34 (VDDD6), C58.2; no longer C37.1, C38.1, C39.1, C40.1, C45.1, C46.1, C47.1, C48.1, U7.19 (VDDD4), U7.37 (VDDD7), U7.43 (VDDA1), U7.46 (VDDA2), U7.49 (VDDA3), U7.5 (VDDD2), U7.52 (VDDA4), U7.70 (VDDD9)
- net +5V: now also C45.1, C46.1, C47.1, C48.1, U7.19 (VDDD4), U7.37 (VDDD7), U7.5 (VDDD2), U7.70 (VDDD9)
- net GND: now also U7.12 (TTX), U7.31 (VSSD6), U7.38 (CDIR), U7.54 (SELI), U7.65 (AP), U7.66 (SP), U7.75 (SA), U7.77 (OVL2), U7.78 (OVL1), U7.79 (OVL0), U7.80 (KEY), C58.1
- net +3V3A2: now reaches C31.1, C32.1, C33.1, C34.1, C35.1, L3.2, U7.56 (VDDA6), U7.58 (VDDA7), U7.60 (VDDA8), U7.62 (VDDA9)
- net +3V3A2: now also C36.1, C37.1, C38.1, C39.1, C40.1, U7.43 (VDDA1), U7.46 (VDDA2), U7.49 (VDDA3), U7.52 (VDDA4), U7.53 (VDDA5)
- no-connect marks 2 -> 7
Other:
- note added: "+3V3 Analog for Encoder"
- note added: "TODO: determine if RTCI should be connected to ground"
- moved on the sheet: C30, C31, L3, R14, R15, R16, R17, R19, R20, R21, R22, R23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

Commit message: minor cleanup, addition of notes
Other:
- note added: "+3V3 Analog LC Filter for Encoder"
- note added: "Refer NOTES (item 4) above"
- note added: "TODO: Unsure on level matching for the LS74, check RCV1 and RCV2 specs and make sure they are ok to drive the flip-flop input and clock."
- note removed: "+3V3 Analog for Encoder"
- moved on the sheet: C27, C28, C29, C30, C31, C32, C33, C34, C35, C36, C37, C38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

Commit message: resistor footprint added
Parts:
- R13, R14, R15, R16, R17, R18, R19, R20, R21, R22, R23, R24, R25, R26: footprint (none) -> tbc:R0603
- U7: footprint (none) -> tbc:QFP80_14x20x2.8mm_Pitch0.8mm
Changed lines of the file:
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@@
       (effects (font (size 1.27 1.27)) (justify right))
     )
-    (property "Footprint" "" (at 248.92 166.37 0)
+    (property "Footprint" "tbc:R0603" (at 248.92 149.86 0) (show_name)
       (effects (font (size 1.27 1.27)) hide)
     )
@@
       (effects (font (size 1.27 1.27)) (justify right))
     )
-    (property "Footprint" "" (at 240.03 166.37 0)
+    (property "Footprint" "tbc:R0603" (at 240.03 149.86 0) (show_name)
       (effects (font (size 1.27 1.27)) hide)
     )
@@
       (effects (font (size 1.27 1.27)) (justify left) hide)
     )
-    (property "Sim.Enable" "0" (at 232.41 149.86 0)
+    (property "Sim.Enable" "0" (at 237.49 149.86 0)
       (effects (font (size 1.27 1.27)) hide)
     )
@@
       (effects (font (size 1.27 1.27)))
     )
-    (property "Footprint" "" (at 190.5 149.86 0)
+    (property "Footprint" "tbc:R0603" (at 207.01 149.86 0) (show_name)
       (effects (font (size 1.27 1.27)) hide)
     )
@@
       (effects (font (size 1.27 1.27)))
     )
-    (property "Footprint" "" (at 190.5 123.19 0)
+    (property "Footprint" "tbc:R0603" (at 207.01 123.19 0) (show_name)
       (effects (font (size 1.27 1.27)) hide)
     )
@@
       (effects (font (size 1.27 1.27)))
     )
-    (property "Footprint" "" (at 190.5 116.84 0)
+    (property "Footprint" "tbc:R0603" (at 207.01 116.84 0) (show_name)
       (effects (font (size 1.27 1.27)) hide)
     )
@@
       (effects (font (size 1.27 1.27)) (justify right))
     )
-    (property "Footprint" "" (at 267.97 166.37 0)
+    (property "Footprint" "tbc:R0603" (at 267.97 149.86 0) (show_name)
       (effects (font (size 1.27 1.27)) hide)
     )
@@
       (effects (font (size 1.27 1.27)) (justify right))
     )
-    (property "Footprint" "" (at 85.09 62.23 0)
+    (property "Footprint" "tbc:R0603" (at 68.58 62.23 0) (show_name)
       (effects (font (size 1.27 1.27)) hide)
     )
@@
       (effects (font (size 1.27 1.27)) (justify right))
     )
-    (property "Footprint" "" (at 259.08 166.37 0)
+    (property "Footprint" "tbc:R0603" (at 259.08 149.86 0) (show_name)
       (effects (font (size 1.27 1.27)) hide)
     )
@@
       (effects (font (size 1.27 1.27)))
     )
-    (property "Footprint" "" (at 106.68 87.63 0)
+    (property "Footprint" "tbc:QFP80_14x20x2.8mm_Pitch0.8mm" (at 140.97 173.99 0) (show_name)
       (effects (font (size 1.27 1.27)) hide)
     )
@@
       (effects (font (size 1.27 1.27)))
     )
-    (property "Footprint" "" (at 190.5 143.51 0)
+    (property "Footprint" "tbc:R0603" (at 207.01 143.51 0) (show_name)
       (effects (font (size 1.27 1.27)) hide)
     )
@@
       (effects (font (size 1.27 1.27)))
     )
-    (property "Footprint" "" (at 190.5 129.54 0)
+    (property "Footprint" "tbc:R0603" (at 207.01 129.54 0) (show_name)
       (effects (font (size 1.27 1.27)) hide)
     )
@@
       (effects (font (size 1.27 1.27)) (justify right))
     )
-    (property "Footprint" "" (at 231.14 166.37 0)
+    (property "Footprint" "tbc:R0603" (at 231.14 149.86 0) (show_name)
       (effects (font (size 1.27 1.27)) hide)
     )
@@
       (effects (font (size 1.27 1.27)) (justify left) hide)
     )
-    (property "Sim.Enable" "0" (at 223.52 149.86 0)
+    (property "Sim.Enable" "0" (at 228.6 149.86 0)
       (effects (font (size 1.27 1.27)) hide)
     )
@@
       (effects (font (size 1.27 1.27)) (justify right))
     )
-    (property "Footprint" "" (at 222.25 166.37 0)
+    (property "Footprint" "tbc:R0603" (at 222.25 149.86 0) (show_name)
       (effects (font (size 1.27 1.27)) hide)
     )
@@
       (effects (font (size 1.27 1.27)))
     )
-    (property "Footprint" "" (at 190.5 137.16 0)
+    (property "Footprint" "tbc:R0603" (at 207.01 137.16 0) (show_name)
       (effects (font (size 1.27 1.27)) hide)
     )
@@
       (effects (font (size 1.27 1.27)) (justify right))
     )
-    (property "Footprint" "" (at 107.95 191.77 0)
-      (effects (font (size 1.27 1.27)) hide)
-    )
+    (property "Footprint" "tbc:R0603" (at 107.95 175.26 0) (show_name)
+      (effects (font (size 1.27 1.27)) hide)
+    )

Commit message: footprints and 3d models for caps, connectors
Parts:
- C27, C28, C29, C30, C32, C33, C34, C35, C36, C37, C38, C39, C40, C41, C42, C43, C44, C45, C46, C47, C48, C49, C58: footprint (none) -> tbc:C0603
Changed lines of the file:
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@@
       (effects (font (size 1.27 1.27)))
     )
-    (property "Footprint" "" (at 170.18 46.99 0)
+    (property "Footprint" "tbc:C0603" (at 170.18 46.99 0)
       (effects (font (size 1.27 1.27)) hide)
     )
@@
       (effects (font (size 1.27 1.27)))
     )
-    (property "Footprint" "" (at 96.52 63.5 0)
+    (property "Footprint" "tbc:C0603" (at 96.52 63.5 0)
       (effects (font (size 1.27 1.27)) hide)
     )
@@
       (effects (font (size 1.27 1.27)))
     )
-    (property "Footprint" "" (at 170.18 62.23 0)
+    (property "Footprint" "tbc:C0603" (at 170.18 62.23 0)
       (effects (font (size 1.27 1.27)) hide)
     )
@@
       (effects (font (size 1.27 1.27)))
     )
-    (property "Footprint" "" (at 147.32 46.99 0)
+    (property "Footprint" "tbc:C0603" (at 147.32 46.99 0)
       (effects (font (size 1.27 1.27)) hide)
     )
@@
       (effects (font (size 1.27 1.27)))
     )
-    (property "Footprint" "" (at 121.92 54.61 0)
+    (property "Footprint" "tbc:C0603" (at 121.92 54.61 0)
       (effects (font (size 1.27 1.27)) hide)
     )
@@
       (effects (font (size 1.27 1.27)))
     )
-    (property "Footprint" "" (at 93.98 180.34 0)
+    (property "Footprint" "tbc:C0603" (at 93.98 180.34 0)
       (effects (font (size 1.27 1.27)) hide)
     )
@@
       (effects (font (size 1.27 1.27)))
     )
-    (property "Footprint" "" (at 170.18 69.85 0)
+    (property "Footprint" "tbc:C0603" (at 170.18 69.85 0)
       (effects (font (size 1.27 1.27)) hide)
     )
@@
       (effects (font (size 1.27 1.27)))
     )
-    (property "Footprint" "" (at 147.32 62.23 0)
+    (property "Footprint" "tbc:C0603" (at 147.32 62.23 0)
       (effects (font (size 1.27 1.27)) hide)
     )
@@
       (effects (font (size 1.27 1.27)) (justify right))
     )
-    (property "Footprint" "" (at 53.34 81.28 0)
+    (property "Footprint" "tbc:C0603" (at 53.34 81.28 0)
       (effects (font (size 1.27 1.27)) hide)
     )
@@
       (effects (font (size 1.27 1.27)))
     )
-    (property "Footprint" "" (at 121.92 62.23 0)
+    (property "Footprint" "tbc:C0603" (at 121.92 62.23 0)
       (effects (font (size 1.27 1.27)) hide)
     )
@@
       (effects (font (size 1.27 1.27)))
     )
-    (property "Footprint" "" (at 254 74.93 0)
+    (property "Footprint" "tbc:C0603" (at 254 74.93 0)
       (effects (font (size 1.27 1.27)) hide)
     )
@@
       (effects (font (size 1.27 1.27)))
     )
-    (property "Footprint" "" (at 170.18 54.61 0)
+    (property "Footprint" "tbc:C0603" (at 170.18 54.61 0)
       (effects (font (size 1.27 1.27)) hide)
     )
@@
       (effects (font (size 1.27 1.27)))
     )
-    (property "Footprint" "" (at 48.26 71.12 0)
+    (property "Footprint" "tbc:C0603" (at 48.26 71.12 0)
       (effects (font (size 1.27 1.27)) hide)
     )
@@
       (effects (font (size 1.27 1.27)))
     )
-    (property "Footprint" "" (at 121.92 46.99 0)
+    (property "Footprint" "tbc:C0603" (at 121.92 46.99 0)
       (effects (font (size 1.27 1.27)) hide)
     )
@@
       (effects (font (size 1.27 1.27)))
     )
-    (property "Footprint" "" (at 147.32 69.85 0)
+    (property "Footprint" "tbc:C0603" (at 147.32 69.85 0)
       (effects (font (size 1.27 1.27)) hide)
     )
@@
       (effects (font (size 1.27 1.27)))
     )
-    (property "Footprint" "" (at 193.04 46.99 0)
+    (property "Footprint" "tbc:C0603" (at 193.04 46.99 0)
       (effects (font (size 1.27 1.27)) hide)
     )
@@
       (effects (font (size 1.27 1.27)))
     )
-    (property "Footprint" "" (at 193.04 54.61 0)
+    (property "Footprint" "tbc:C0603" (at 193.04 54.61 0)
       (effects (font (size 1.27 1.27)) hide)
     )
@@
       (effects (font (size 1.27 1.27)))
     )
-    (property "Footprint" "" (at 48.26 58.42 0)
+    (property "Footprint" "tbc:C0603" (at 48.26 58.42 0)
       (effects (font (size 1.27 1.27)) hide)
     )
@@
       (effects (font (size 1.27 1.27)))
     )
-    (property "Footprint" "" (at 121.92 69.85 0)
+    (property "Footprint" "tbc:C0603" (at 121.92 69.85 0)
       (effects (font (size 1.27 1.27)) hide)
     )
@@
       (effects (font (size 1.27 1.27)))
     )
-    (property "Footprint" "" (at 147.32 39.37 0)
+    (property "Footprint" "tbc:C0603" (at 147.32 39.37 0)
       (effects (font (size 1.27 1.27)) hide)
     )
@@
       (effects (font (size 1.27 1.27)))
     )
-    (property "Footprint" "" (at 193.04 69.85 0)
+    (property "Footprint" "tbc:C0603" (at 193.04 69.85 0)
       (effects (font (size 1.27 1.27)) hide)
     )
@@
       (effects (font (size 1.27 1.27)))
     )
-    (property "Footprint" "" (at 193.04 62.23 0)
+    (property "Footprint" "tbc:C0603" (at 193.04 62.23 0)
       (effects (font (size 1.27 1.27)) hide)
     )
@@
       (effects (font (size 1.27 1.27)))
     )
-    (property "Footprint" "" (at 147.32 54.61 0)
-      (effects (font (size 1.27 1.27)) hide)
-    )
+    (property "Footprint" "tbc:C0603" (at 147.32 54.61 0)
+      (effects (font (size 1.27 1.27)) hide)
+    )

Commit message: initial work on layout
Parts:
- U8: value SN74LS74ADR -> CD74HC74M96; footprint (none) -> tbc:SOIC-14; symbol tbc:SN74LS74ADR -> tbc:CD74HC74M96; Mouser 595-SN74LS74ADR -> 595-CD74HC74M96
Changed lines of the file:
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@@
     )
   )
-  (symbol (lib_id "tbc:SN74LS74ADR") (at 241.3 82.55 0) (unit 1)
+  (symbol (lib_id "tbc:CD74HC74M96 ") (at 241.3 82.55 0) (unit 1)
     (in_bom yes) (on_board yes) (dnp no)
     (property "Reference" "U8" (at 232.41 66.04 0)
       (effects (font (size 1.27 1.27)) (justify left))
     )
-    (property "Value" "SN74LS74ADR" (at 246.38 99.06 0)
-      (effects (font (size 1.27 1.27)) (justify left))
+    (property "Value" "CD74HC74M96 " (at 251.46 99.06 0)
+      (effects (font (size 1.27 1.27)))
     )
-    (property "Footprint" "" (at 229.87 76.2 0)
+    (property "Footprint" "tbc:SOIC-14" (at 241.3 119.38 0) (show_name)
       (effects (font (size 1.27 1.27)) hide)
     )
-    (property "Datasheet" "https://www.ti.com/lit/ds/symlink/sn54s74.pdf?ts=1706174643586&ref_url=https%253A%252F%252Fau.mouser.com%252F" (at 242.57 111.76 0) (show_name)
+    (property "Datasheet" "https://www.ti.com/lit/gpn/cd74hc74" (at 242.57 111.76 0) (show_name)
       (effects (font (size 1.27 1.27)) hide)
     )
-    (property "Mouser" " 595-SN74LS74ADR" (at 241.3 114.3 0) (show_name)
+    (property "Mouser" " 595-CD74HC74M96 " (at 241.3 114.3 0) (show_name)
       (effects (font (size 1.27 1.27)) hide)
     )
-    (property "Sim.Enable" "0" (at 241.3 82.55 0)
+    (property "Sim.Enable" "0" (at 241.3 116.84 0) (show_name)
       (effects (font (size 1.27 1.27)) hide)
     )

Commit message: added footprints for crystals and updated layout
Parts:
- Y1: footprint (none) -> tbc:ABLS
Changed lines of the file:
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@@
       (effects (font (size 0.635 0.635)) hide)
     )
-    (property "Footprint" "" (at 72.39 76.2 0)
+    (property "Footprint" "tbc:ABLS" (at 72.39 76.2 0)
       (effects (font (size 1.27 1.27)) hide)
     )
