File: encoder.kicad_sch (KiCad schematic)
At the start: 43 parts, among them U7 SAA7182A, U8 CD74HC74M96, Y1 ABLS-27.000MHZ-B2F-T

Commit message: 3V3A component footprints + layout work
Parts:
- L3: footprint (none) -> tbc:DFE201610E
Changed lines of the file:
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@@
       (effects (font (size 1.27 1.27)))
     )
-    (property "Footprint" "" (at 41.91 168.91 90)
+    (property "Footprint" "tbc:DFE201610E" (at 41.91 168.91 90)
       (effects (font (size 1.27 1.27)) hide)
     )

Commit message: layout LHS
Parts:
- C31: footprint (none) -> tbc:GRM32
Changed lines of the file:
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@@
       (effects (font (size 1.27 1.27)))
     )
-    (property "Footprint" "" (at 39.37 175.26 0)
+    (property "Footprint" "tbc:GRM32" (at 39.37 175.26 0)
       (effects (font (size 1.27 1.27)) hide)
     )

Commit message: layout complete and passed DRC
Parts:
- L2: footprint (none) -> tbc:L0805
Changed lines of the file:
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@@
       (effects (font (size 1.27 1.27)))
     )
-    (property "Footprint" "" (at 43.18 92.71 90)
+    (property "Footprint" "tbc:L0805" (at 43.18 92.71 90)
       (effects (font (size 1.27 1.27)) hide)
     )

Commit message: updates from library, performed ERC/DRC, update Kicad 8.0.8
Parts:
- U8: value CD74HC74M96 -> CD74HC74M96
Changed lines of the file:
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@@
 	(label "DP2"
 		(at 72.39 101.6 0)
-		(fields_autoplaced yes)
 		(effects
 			(font
@@
 	(label "MP3"
 		(at 72.39 121.92 0)
-		(fields_autoplaced yes)
 		(effects
 			(font
@@
 	(label "MP5"
 		(at 72.39 116.84 0)
-		(fields_autoplaced yes)
 		(effects
 			(font
@@
 	(label "MP1"
 		(at 72.39 127 0)
-		(fields_autoplaced yes)
 		(effects
 			(font
@@
 	(label "DP5"
 		(at 72.39 93.98 0)
-		(fields_autoplaced yes)
 		(effects
 			(font
@@
 	(label "MP4"
 		(at 72.39 119.38 0)
-		(fields_autoplaced yes)
 		(effects
 			(font
@@
 	(label "DP6"
 		(at 72.39 91.44 0)
-		(fields_autoplaced yes)
 		(effects
 			(font
@@
 	(label "MP0"
 		(at 72.39 129.54 0)
-		(fields_autoplaced yes)
 		(effects
 			(font
@@
 	(label "DP1"
 		(at 72.39 104.14 0)
-		(fields_autoplaced yes)
 		(effects
 			(font
@@
 	(label "MP2"
 		(at 72.39 124.46 0)
-		(fields_autoplaced yes)
 		(effects
 			(font
@@
 	(label "DP3"
 		(at 72.39 99.06 0)
-		(fields_autoplaced yes)
 		(effects
 			(font
@@
 	(label "MP6"
 		(at 72.39 114.3 0)
-		(fields_autoplaced yes)
 		(effects
 			(font
@@
 	(label "MP7"
 		(at 72.39 111.76 0)
-		(fields_autoplaced yes)
 		(effects
 			(font
@@
 	(label "DP4"
 		(at 72.39 96.52 0)
-		(fields_autoplaced yes)
 		(effects
 			(font
@@
 	(label "DP0"
 		(at 72.39 106.68 0)
-		(fields_autoplaced yes)
 		(effects
 			(font
@@
 	(label "DP7"
 		(at 72.39 88.9 0)
-		(fields_autoplaced yes)
 		(effects
 			(font
@@
 		(shape output)
 		(at 213.36 92.71 270)
-		(fields_autoplaced yes)
 		(effects
 			(font
@@
 		(shape output)
 		(at 264.16 142.24 0)
-		(fields_autoplaced yes)
 		(effects
 			(font
@@
 		(shape input)
 		(at 67.31 133.35 180)
-		(fields_autoplaced yes)
 		(effects
 			(font
@@
 		(shape output)
 		(at 199.39 91.44 0)
-		(fields_autoplaced yes)
 		(effects
 			(font
@@
 		(shape output)
 		(at 264.16 109.22 0)
-		(fields_autoplaced yes)
 		(effects
 			(font
@@
 		(shape input)
 		(at 102.87 168.91 0)
-		(fields_autoplaced yes)
 		(effects
 			(font
@@
 		(shape input)
 		(at 76.2 139.7 180)
-		(fields_autoplaced yes)
 		(effects
 			(font
@@
 		(shape output)
 		(at 256.54 92.71 0)
-		(fields_autoplaced yes)
 		(effects
 			(font
@@
 		(shape output)
 		(at 264.16 121.92 0)
-		(fields_autoplaced yes)
 		(effects
 			(font
@@
 		(shape output)
 		(at 199.39 81.28 0)
-		(fields_autoplaced yes)
 		(effects
 			(font
@@
 		(shape output)
 		(at 256.54 85.09 0)
-		(fields_autoplaced yes)
 		(effects
 			(font
@@
 		(shape output)
 		(at 264.16 129.54 0)
-		(fields_autoplaced yes)
 		(effects
 			(font
@@
 		(shape output)
 		(at 264.16 115.57 0)
-		(fields_autoplaced yes)
 		(effects
 			(font
@@
 		(shape output)
 		(at 264.16 135.89 0)
-		(fields_autoplaced yes)
 		(effects
 			(font
@@
 		(shape output)
 		(at 210.82 92.71 270)
-		(fields_autoplaced yes)
 		(effects
 			(font
@@
 		(shape input)
 		(at 67.31 110.49 180)
-		(fields_autoplaced yes)
 		(effects
 			(font
@@
 		(shape bidirectional)
 		(at 76.2 142.24 180)
-		(fields_autoplaced yes)
 		(effects
 			(font
@@
 			)
 		)
+		(property "Sim.Enable" "0"
+			(at 105.41 200.406 0)
+			(effects
+				(font
+					(size 1.27 1.27)
+				)
+				(hide yes)
+			)
+		)
 		(pin "1"
 		)
@@
 			)
 		)
+		(property "Sim.Enable" "0"
+			(at 101.6 61.976 0)
+			(effects
+				(font
+					(size 1.27 1.27)
+				)
+				(hide yes)
+			)
+		)
 		(pin "1"
 		)
@@
 			)
 		)
+		(property "Sim.Enable" "0"
+			(at 33.02 178.816 0)
+			(effects
+				(font
+					(size 1.27 1.27)
+				)
+				(hide yes)
+			)
+		)
 		(pin "1"
 		)
@@
 			)
 		)
-		(property "Value" "CD74HC74M96 "
+		(property "Value" "CD74HC74M96"
 			(at 251.46 99.06 0)
 			(effects
@@
 			(effects
 				(font
+					(size 1.27 1.27)
+				)
+				(hide yes)
+			)
+		)
+		(property "Sim.Enable" "0"
+			(at 163.83 42.926 0)
+			(effects
+				(font
