File: tbc.kicad_pcb (KiCad board)
At the start: 4 copper layers, 180 x 67 mm, 130 parts, among them J1 5749181-1, J2 PJRAN1X1U01X, J3 PJRAN1X1U01X, J4 5749181-1, J5 PJRAN1X1U01X, J6 PJRAN3X1U03X, J7 4840.2201, J8 20021111-00010T4LF, J9 75869-105LF, Q1 BSS308PE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

Commit message: added copper pours to layers
Routing:
- net GND: track 277.9 -> 278.9 mm, vias 127 -> 198
- net +5V: vias 31 -> 30
- net +3V3: vias 32 -> 31
- added copper zone on In2.Cu, net GND
